Commit message: refactor: add base_footprint link for odom

File: ucrbot/urdf/ucrbot.urdf (robot description, URDF)
Before this commit: robot ucrbot, 7 links, 6 joints
Links:
- added link base_footprint; visual box size=0.001 0.001 0.001
Joints:
- added joint base_footprint_joint: type fixed, parent base_footprint, child base_link, origin xyz=-0.64 0 -0.04 rpy=0 0 1.5708

Commit message: fix: modify ucrbot.urdf

File: ucrbot/urdf/ucrbot.urdf (robot description, URDF)
Before this commit: robot ucrbot, 7 links, 6 joints
Links:
- link base_link: mass 5.8428 -> 5.84279395822244
- link front_holder: mass 2.406 -> 2.40596398964761
- link front_left_wheel: mass 3.4015 -> 3.40151426652415
- link front_right_wheel: mass 2.9947 -> 2.99473805676772
- link rear_holder: mass 2.0894 -> 2.0893671403394
- link rear_wheel: mass 6.3963 -> 6.39625232328686
Joints:
- joint front_left_drive_joint: origin xyz=0 -0.05 0 rpy=-0.82552 5.3169E-16 4.9093E-16 -> xyz=0 -0.111599999999999 0 rpy=-0.825519933902369 5.29090660172926E-16 4.88758339356465E-16
- joint front_right_drive_joint: origin xyz=0.030426 -0.1116 0 rpy=0.48282 4.3368E-17 -8.3917E-17 -> xyz=0.0304259917277344 -0.1116 0 rpy=0.482824124437366 4.77048955893622E-17 -9.41087485717418E-17
- joint rear_drive_joint: origin xyz=0 -0.0069725 0.14017 rpy=2.3423 -1.8041E-16 1.1506E-15 -> xyz=0 0 0.133000000000013 rpy=2.34234748597585 -1.80411241501588E-16 1.15055534544162E-15
- joint rear_holder_joint: origin xyz=0 -0.09 -0.1116 rpy=1.5708 -0.0025759 1.5772E-19 -> xyz=0 -0.0899999999999911 -0.1116 rpy=1.5707963267949 -0.00257589519748985 1.57723230125107E-19

Commit message: fix: add velocity limit into ucrbot.urdf for steering control in gazebo

File: ucrbot/urdf/ucrbot.urdf (robot description, URDF)
Before this commit: robot ucrbot, 7 links, 6 joints
Joints:
- joint front_steer_joint: limit lower=-0.5 upper=0.5 effort=0 velocity=0 -> lower=-0.5 upper=0.5 effort=0 velocity=1
