Commit message: refactor: modify ucr_epos_control package for new ucrbot.urdf

File: ucr_description/urdf/xacro/transmissions.xacro (robot description, xacro)
@@ -2,20 +2,20 @@
 <robot name="ucrbot" xmlns:xacro="http://www.ros.org/wiki/xacro">
     <!-- transmission of steer drive -->
-    <transmission name="steer_joint_trans" >
+    <transmission name="front_steer_joint_trans" >
         <type>transmission_interface/SimpleTransmission</type>
-        <joint name="steer_joint" >
+        <joint name="front_steer_joint" >
             <hardwareInterface>hardware_interface/PositionJointInterface</hardwareInterface>
         </joint>
-        <actuator name="steer_actuator" >
+        <actuator name="front_steer_actuator" >
             <mechanicalReduction>200</mechanicalReduction>
         </actuator>
     </transmission>
     <!-- transmission of rear wheel -->
-    <transmission name="rear_left_drive_joint_trans" >
+    <transmission name="rear_drive_joint_trans" >
         <type>transmission_interface/SimpleTransmission</type>
-        <joint name="rear_left_drive_joint" >
+        <joint name="rear_drive_joint" >
             <hardwareInterface>hardware_interface/VelocityJointInterface</hardwareInterface>
         </joint>
-        <actuator name="rear_left_drive_actuator" >
+        <actuator name="rear_drive_actuator" >
             <mechanicalReduction>244</mechanicalReduction>
         </actuator>

File: ucrbot/urdf/ucrbot.urdf (robot description, URDF)
Before this commit: robot ucrbot, 8 links, 7 joints
Links:
- removed link rear_left_wheel
- removed link rear_right_wheel
- added link rear_wheel, mass 6.3963; collision mesh filename=package://ucrbot/meshes/rear_wheel.STL; visual mesh filename=package://ucrbot/meshes/rear_wheel.STL
- link base_link: mass 7.17075879708735 -> 5.8428
- link front_holder: mass 2.95565551037739 -> 2.406
- link front_left_wheel: mass 2.96434014657607 -> 3.4015
- link front_right_wheel: mass 2.96434014657607 -> 2.9947
- link rear_holder: mass 2.62485787651341 -> 2.0894
Joints:
- removed joint rear_left_drive_joint
- removed joint rear_right_drive_joint
- removed joint rear_rolling_joint
- removed joint steer_joint
- added joint front_steer_joint: type revolute, parent base_link, child front_holder, origin xyz=0 0.145 0 rpy=1.5708 -2.5737E-19 -0.0042033, axis 0 1 0, limit lower=-0.5 upper=0.5 effort=0 velocity=0
- added joint rear_drive_joint: type continuous, parent rear_holder, child rear_wheel, origin xyz=0 -0.0069725 0.14017 rpy=2.3423 -1.8041E-16 1.1506E-15, axis 1 0 0
- added joint rear_holder_joint: type continuous, parent base_link, child rear_holder, origin xyz=0 -0.09 -0.1116 rpy=1.5708 -0.0025759 1.5772E-19, axis 0 0 1
- joint base_footprint_joint: origin xyz=-0.64 0 -0.04 rpy=0 0 1.5708 -> xyz=0 0 0 rpy=0 0 -1.5708
- joint front_left_drive_joint: axis -1 0 0 -> 1 0 0; origin xyz=-0.0325001601438198 -0.0614618553961881 0 rpy=3.14159265358979 4.33680868994202E-19 3.14159265358979 -> xyz=0 -0.05 0 rpy=-0.82552 5.3169E-16 4.9093E-16
- joint front_right_drive_joint: origin xyz=0.0325001601436291 -0.0614618553960491 0 rpy=0 0 0 -> xyz=0.030426 -0.1116 0 rpy=0.48282 4.3368E-17 -8.3917E-17

Commit message: fix: modify transmissiont context in urdf

File: ucr_description/urdf/xacro/transmissions.xacro (robot description, xacro)
@@ -1,4 +1,12 @@
 <?xml version="1.0"?>
 <robot name="ucrbot" xmlns:xacro="http://www.ros.org/wiki/xacro">
+    <!-- macro for mechanical reduction
+    default unit of position motor is qc/s
+    default unit of velocity motor is rmp -->
+    <xacro:property name="PI" value="3.141592653" />
+    <xacro:property name="std2rpm_rate" value="${30/PI}" />
+    <xacro:property name="steer_encoder_resolution" value="2000" />
+    <xacro:property name="steer_gear_reduction" value="200" />
+    <xacro:property name="drive_gear_reduction" value="244" />
     <!-- transmission of steer drive -->
     <transmission name="front_steer_joint_trans" >
@@ -8,5 +16,7 @@
         </joint>
         <actuator name="front_steer_actuator" >
-            <mechanicalReduction>200</mechanicalReduction>
+            <mechanicalReduction>
+                ${steer_gear_reduction*steer_encoder_resolution/2/PI}
+            </mechanicalReduction>
         </actuator>
     </transmission>
@@ -18,5 +28,7 @@
         </joint>
         <actuator name="rear_drive_actuator" >
-            <mechanicalReduction>244</mechanicalReduction>
+            <mechanicalReduction>
+                ${drive_gear_reduction*std2rpm_rate}
+            </mechanicalReduction>
         </actuator>
     </transmission>

Commit message: chore

File: ucr_description/urdf/xacro/transmissions.xacro (robot description, xacro)
@@ -5,5 +5,5 @@
     default unit of velocity motor is rmp -->
     <xacro:property name="PI" value="3.141592653" />
-    <xacro:property name="std2rpm_rate" value="${30/PI}" />
+    <xacro:property name="std2rpm_ratio" value="${30/PI}" />
     <xacro:property name="steer_encoder_resolution" value="2000" />
     <xacro:property name="steer_gear_reduction" value="200" />
@@ -29,5 +29,5 @@
         <actuator name="rear_drive_actuator" >
             <mechanicalReduction>
-                ${drive_gear_reduction*std2rpm_rate}
+                ${drive_gear_reduction*std2rpm_ratio}
             </mechanicalReduction>
         </actuator>

Commit message: feat: run steer_drive_controller together with front_left_wheel_follow_controller in ucr_gazebo_control package; modify axis direction of wheels; rename ucr_steer_drive_control to ucr_control and add full-stack launch file

File: ucr_description/urdf/xacro/transmissions.xacro (robot description, xacro)
@@ -33,3 +33,15 @@
         </actuator>
     </transmission>
+    <!-- transmission of front left wheel -->
+    <transmission name="front_left_joint_trans" >
+        <type>transmission_interface/SimpleTransmission</type>
+        <joint name="front_left_drive_joint" >
+            <hardwareInterface>hardware_interface/VelocityJointInterface</hardwareInterface>
+        </joint>
+        <actuator name="front_left_drive_actuator" >
+            <mechanicalReduction>
+                ${drive_gear_reduction*std2rpm_ratio}
+            </mechanicalReduction>
+        </actuator>
+    </transmission>
 </robot>

File: ucrbot/urdf/ucrbot.urdf (robot description, URDF)
Before this commit: robot ucrbot, 7 links, 6 joints
Links:
- added link camera
- added link imu
Joints:
- added joint camera_joint: type fixed, parent base_link, child camera, origin xyz=0 0 0.1286 rpy=0 0 0
- added joint imu_joint: type fixed, parent base_link, child imu, origin xyz=-0.024 0.15475 0.1039 rpy=0 0 0
- joint base_footprint_joint: origin xyz=0 0 0 rpy=0 0 -1.5708 -> xyz=0.223 -0.001 0.1116 rpy=0 0 -1.5708
- joint front_left_drive_joint: axis 1 0 0 -> -1 0 0
- joint front_right_drive_joint: axis 1 0 0 -> -1 0 0
- joint rear_drive_joint: axis 1 0 0 -> -1 0 0

Commit message: refactor: 1, merger the start up of steer_drive_controller and front_left_drive_controller; 2,delete duplicated launch together with their config in ucr_gazebo_control; 3, rename front_left_wheel_follow_controller to front_left_wheel_autodrive; 4, make launch of HWSim/HW(epos.launch or ucrbot_gazebo_xxx_world.launch), control(ucr_control/launch or ucr_gazebo_control/launch) and teleop functions independently.

File: ucr_description/urdf/xacro/transmissions.xacro (robot description, xacro)
@@ -4,8 +4,9 @@
     default unit of position motor is qc/s
     default unit of velocity motor is rmp -->
-    <xacro:property name="PI" value="3.141592653" />
-    <xacro:property name="std2rpm_ratio" value="${30/PI}" />
-    <xacro:property name="steer_encoder_resolution" value="2000" />
+    <xacro:property name="M_PI" value="3.141592653" />
+    <xacro:property name="std2rpm_ratio" value="${30/M_PI}" />
+    <xacro:property name="steer_encoder_quadcounter" value="4096" />
     <xacro:property name="steer_gear_reduction" value="200" />
+    <xacro:property name="drive_encoder_quadcounter" value="4000" />
     <xacro:property name="drive_gear_reduction" value="244" />
     <!-- transmission of steer drive -->
@@ -17,5 +18,5 @@
         <actuator name="front_steer_actuator" >
             <mechanicalReduction>
-                ${steer_gear_reduction*steer_encoder_resolution/2/PI}
+                ${steer_gear_reduction*steer_encoder_quadcounter/2/M_PI}
             </mechanicalReduction>
         </actuator>
