Commit message: feat: rename original base_footprint to odom_link and add new base_footprint

File: ucr_gazebo/urdf/transmissions_steer_bot_hardware.xacro (robot description, xacro)
@@ -11,5 +11,5 @@
     <xacro:property name="drive_gear_reduction" value="244" />
     <!-- transmission of steer drive -->
-    <!--transmission name="front_steer_joint_trans" >
+    <transmission name="front_steer_joint_trans" >
         <type>transmission_interface/SimpleTransmission</type>
         <joint name="front_steer_joint" >
@@ -21,5 +21,5 @@
             </mechanicalReduction>
         </actuator>
-    </transmission-->
+    </transmission>
     <!-- transmission of rear wheel -->
     <transmission name="rear_drive_joint_trans" >
@@ -38,5 +38,5 @@
         <type>transmission_interface/SimpleTransmission</type>
         <joint name="front_left_drive_joint" >
-            <hardwareInterface>EffortJointInterface</hardwareInterface>
+            <hardwareInterface>hardware_interface/VelocityJointInterface</hardwareInterface>
         </joint>
         <actuator name="front_left_drive_actuator" >
@@ -46,3 +46,15 @@
         </actuator>
     </transmission>
+    <!-- transmission of front right wheel -->
+    <transmission name="front_right_joint_trans" >
+        <type>transmission_interface/SimpleTransmission</type>
+        <joint name="front_right_drive_joint" >
+            <hardwareInterface>hardware_interface/VelocityJointInterface</hardwareInterface>
+        </joint>
+        <actuator name="front_right_drive_actuator" >
+            <mechanicalReduction>
+                ${drive_gear_reduction*std2rpm_ratio}
+            </mechanicalReduction>
+        </actuator>
+    </transmission>
 </robot>

File: ucr_gazebo/urdf/ucrbot.gazebo.xacro (robot description, xacro)
@@ -23,3 +23,6 @@
     <fdir1 value="1 0 0"/>
   </gazebo>
+  <gazebo reference="base_link">
+    <gravity value="true" />
+  </gazebo>
 </robot>

File: ucrbot/urdf/ucrbot.urdf (robot description, URDF)
Before this commit: robot ucrbot, 9 links, 8 joints
Links:
- added link odom_link
- link base_footprint: geometry 
Joints:
- added joint odom_joint: type fixed, parent odom_link, child base_link, origin xyz=0.223 -0.001 0.1116 rpy=0 0 -1.5708
- joint base_footprint_joint: child base_link -> odom_link; origin xyz=0.223 -0.001 0.1116 rpy=0 0 -1.5708 -> xyz=-0.1575 0 0 rpy=0 0 0
