Commit message: add ucr_ekf package and modify manner of rear_holder_joint. Add ucr_ekf which actually runs robot_pose_ekf, and modify the friction param of wheels Make rear holder joint fixed; Fix missing tf(base_link --> base_footprint and base_link --> rear_holder)

File: ucr_gazebo/urdf/description.gazebo.xacro (robot description, xacro)
@@ -5,10 +5,10 @@
   <xacro:include filename="$(find ucr_gazebo)/urdf/ucrbot.gazebo.xacro" />
   <!-- Gazebo plugin for ROS Control -->
-  <!--gazebo>
+  <!-- <gazebo>
     <plugin name="gazebo_ros_control" filename="libgazebo_ros_control.so">
       <robotNamespace>/</robotNamespace>
       <robotSimType>gazebo_ros_control/DefaultRobotHWSim</robotSimType>
     </plugin>
-  </gazebo-->
+  </gazebo> -->
   <gazebo>
     <plugin name="gazebo_ros_control" filename="libgazebo_ros_control.so">
@@ -17,3 +17,22 @@
     </plugin>
   </gazebo>
+  <gazebo reference="imu">
+    <gravity>true</gravity>
+    <sensor name="imu_sensor" type="imu">
+      <always_on>true</always_on>
+      <update_rate>100</update_rate>
+      <visualize>true</visualize>
+      <topic>imu_data</topic>
+      <plugin filename="libgazebo_ros_imu_sensor.so" name="imu_plugin">
+        <topicName>imu_data</topicName>
+        <bodyName>imu</bodyName>
+        <updateRateHZ>10.0</updateRateHZ>
+        <gaussianNoise>0.0</gaussianNoise>
+        <xyzOffset>0 0 0</xyzOffset>
+        <rpyOffset>0 0 0</rpyOffset>
+        <frameName>imu</frameName>
+      </plugin>
+      <pose>0 0 0 0 0 0</pose>
+    </sensor>
+  </gazebo>
 </robot>

File: ucr_gazebo/urdf/ucrbot.gazebo.xacro (robot description, xacro)
@@ -3,6 +3,6 @@
   <gazebo reference="front_left_wheel">
     <!--Friction coefficients-->
-    <mu1 value="5.0"/>
-    <mu2 value="5.0"/>
+    <mu1 value="50.0"/>
+    <mu2 value="50.0"/>
     <kp value="10000000.0" />
     <kd value="1.0" />
@@ -10,6 +10,6 @@
   </gazebo>
   <gazebo reference="front_right_wheel">
-    <mu1 value="5.0"/>
-    <mu2 value="5.0"/>
+    <mu1 value="50.0"/>
+    <mu2 value="50.0"/>
     <kp value="10000000.0" />
     <kd value="1.0" />
@@ -17,6 +17,6 @@
   </gazebo>
   <gazebo reference="rear_wheel">
-    <mu1 value="5.0"/>
-    <mu2 value="5.0"/>
+    <mu1 value="50.0"/>
+    <mu2 value="50.0"/>
     <kp value="10000000.0" />
     <kd value="1.0" />

File: ucrbot/urdf/ucrbot.urdf (robot description, URDF)
Before this commit: robot ucrbot, 10 links, 9 joints
Joints:
- joint rear_holder_joint: axis 0 0 1 -> (none); type continuous -> fixed
