Commit message: modifications. Tune covariance matrix of steer drive controller(gazebo); Disable ackerman link in hardware config(gazebo); Deprecate declaration of gravity in xacro(gazebo); Put base_footprint at odom_link.

File: ucr_gazebo/urdf/ucrbot.gazebo.xacro (robot description, xacro)
@@ -23,6 +23,6 @@
     <fdir1 value="1 0 0"/>
   </gazebo>
-  <gazebo reference="base_link">
+  <!-- <gazebo reference="base_link">
     <gravity value="true" />
-  </gazebo>
+  </gazebo> -->
 </robot>

File: ucrbot/urdf/ucrbot.urdf (robot description, URDF)
Before this commit: robot ucrbot, 10 links, 9 joints
Joints:
- joint base_footprint_joint: origin xyz=-0.1575 0 0 rpy=0 0 0 -> xyz=0 0 0 rpy=0 0 0
